Commit message: manual graph bug

File: urdf/bin-picking-part.urdf (robot description, URDF)
Before this commit: robot bin, 1 links, 0 joints
Links:
- added link handle_link
Joints:
- added joint handle_jonit: type fixed, parent base_link, child handle_link, origin xyz=0.05 0.1 0.015 rpy=0 1.5707963 0

File: urdf/box.urdf (robot description, URDF)
Before this commit: robot box, 1 links, 0 joints
Links:
- added link box_link
- link world: geometry collision box size=0.01 0.8 0.095; collision box size=0.01 0.8 0.095
Joints:
- added joint box_jonit: type fixed, parent world, child box_link, origin xyz=0.86 0.0 0.21 rpy=0 0 0

File: urdf/ur10_bin-picking_sim.urdf.xacro (robot description, xacro)
@@ -51,19 +51,4 @@
          izz="0.001" />
      </inertial>
-     <visual>
-       <origin xyz="0 0 0" rpy="0 0 0" />
-       <geometry>
-         <mesh filename="package://agimus_demos/meshes/ur10e_d435_mount.stl"/>
-       </geometry>
-       <material name="Red">
-         <color rgba="0.9 0.1 0.1 1.0"/>
-       </material>
-     </visual>
-     <collision>
-       <origin xyz="0 0 0" rpy="0 0 0" />
-       <geometry>
-         <mesh filename="package://agimus_demos/meshes/ur10e_d435_mount.stl"/>
-       </geometry>
-     </collision>
    </link>
    <joint name="ur10e_d435_mount_joint" type="fixed">
@@ -117,8 +102,3 @@
 	     rpy="-0.00127120646 -1.00435876 -1.56137241"/>
    </joint>
-   <xacro:include filename="$(find realsense2_description)/urdf/_d435.urdf.xacro" />
-   <xacro:sensor_d435 parent="ref_camera_link" name="camera" use_nominal_extrinsics="true">
-     <!-- <origin xyz="0 0.115 0" rpy="0 -1.0472 -1.57079632679"/> -->
-      <origin xyz="0 0 0" rpy="0 0 0"/>
-   </xacro:sensor_d435>
 </robot>
