Commit message: change support size

File: urdf/additional.urdf.xacro (robot description, xacro)
@@ -16,4 +16,11 @@
      <origin xyz="-1.4 0.0 0.0" rpy="0.0 0.0 0.0" />
    </joint>
+  <joint name="cam_joint" type="fixed">
+     <parent link="world" />
+     <child link = "cam_link" />
+     <origin xyz="0.86 0.0 0.295" rpy="0.0 0.0 -1.5707" />
+  </joint>
+   <link name="cam_link">
+   </link>
     <link name="support_link">
       <inertial>
@@ -23,13 +30,13 @@
       </inertial>
       <visual>
-        <origin xyz="-0.4 0 0.3"/>
+        <origin xyz="-0.4 0 0.25"/>
         <geometry>
-	        <box size="1.0 1.2 0.6"/>
+	        <box size="1.0 1.2 0.5"/>
         </geometry>
       </visual>
       <collision>
-        <origin xyz="-0.4 0 0.3"/>
+        <origin xyz="-0.4 0 0.25"/>
         <geometry>
-	        <box size="1.0 1.2 0.6"/>
+	        <box size="1.0 1.2 0.5"/>
         </geometry>
       </collision>
@@ -43,5 +50,5 @@
       <parent link="support_link" />
       <child link = "base_link" />
-      <origin xyz="0.0 0.0 0.60" rpy="0.0 0.0 -1.5707963" />
+      <origin xyz="0.0 0.0 0.50" rpy="0.0 0.0 -1.5707963" />
     </joint>
   </xacro:macro>
