Commit message: change the size of lid

File: urdf/lip.urdf (robot description, URDF)
Before this commit: robot lip, 1 links, 0 joints
Links:
- link world: geometry collision box size=0.52 0.82 0.002; visual box size=0.52 0.82 0.002

Commit message: update InState Planner Path alg

File: urdf/lip.urdf (robot description, URDF)
Before this commit: robot lip, 1 links, 0 joints
Links:
- link world: geometry collision box size=0.52 0.82 0.002
